File: KiCad_PCB_Example_x/KiCad_PCB_Example_x.kicad_sch (KiCad schematic)
At the start: 0 parts

Commit message: adding resistors
Parts:
- added R1, R2: R, symbol Device:R
Connections:
- new net: R1.2, R2.1
- new net GND: R1.1, R2.2

Commit message: Part 3
Parts:
- removed R1, R2: R, symbol Device:R
- added BT1: 3V, Battery:BatteryHolder_Keystone_1058_1x2032, symbol Device:Battery_Cell
- added D1: RED, LED_THT:LED_D5.0mm, symbol Device:LED
- added R3: 1k, Resistor_THT:R_Axial_DIN0309_L9.0mm_D3.2mm_P12.70mm_Horizontal, symbol Device:R_US
Connections:
- net GND: now also BT1.2 (-), D1.1 (K)
- new net: D1.2 (A), R3.2
- new net VCC: BT1.1 (+), R3.1
