File: KiCad_PCB_Example_x/KiCad_PCB_Example_x.kicad_pcb (KiCad board)
At the start: 2 copper layers, 40.6 x 50 mm, 3 parts

Commit message: Added Initial
Other:
- board text added: "NP"
Changed lines of the file:
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@@
 		(layer "Edge.Cuts")
+	)
+	(gr_text "NP\n"
+		(at 80 57 0)
+		(layer "F.SilkS")
+		(effects
+			(font
+				(size 5 5)
+				(thickness 0.1)
+			)
+			(justify left bottom)
+		)
 	)
 	(segment
